File: cube.sch (EAGLE design)
At the start: 0 parts

Commit message: 1st layer
Parts:
- added C1, C2, C3, C4, C5, C6, C7, C8: 100n, rcl:C-EU050-024X044
- added D1, D10, D11, D12, D13, D14, D15, D16, D17, D18, D19, D2, D20, D21, D22, D23, D24, D25, D26, D27, D28, D29, D3, D30, D31, D32, D33, D34, D35, D36, D37, D38, D39, D4, D40, D41, D42, D43, D44, D45, D46, D47, D48, D49, D5, D50, D51, D52, D53, D54, D55, D56, D57, D58, D59, D6, D60, D61, D62, D63, D64, D7, D8, D9: CLEAR, SparkFun-LED:LED-RGB-CCCLEAR
- added IC1, IC2, IC3, IC4, IC5, IC6, IC7, IC8: TPIC6B595N, tpic:TPIC6B596N
Connections:
- new net GND: C1.2, C2.2, C3.2, C4.2, C5.2, C6.2, C7.2, C8.2, IC1G$1.G, IC2G$1.G, IC3G$1.G, IC4G$1.G, IC5G$1.G, IC6G$1.G, IC7G$1.G, IC8G$1.G
- new net N$1: D1.RED, D10.RED, D11.RED, D12.RED, D13.RED, D14.RED, D15.RED, D16.RED, D17.RED, D18.RED, D19.RED, D2.RED, D20.RED, D21.RED, D22.RED, D23.RED, D24.RED, D25.RED, D26.RED, D27.RED, D28.RED, D29.RED, D3.RED, D30.RED, D31.RED, D32.RED, D33.RED, D34.RED, D35.RED, D36.RED, D37.RED, D38.RED, D39.RED, D4.RED, D40.RED, D41.RED, D42.RED, D43.RED, D44.RED, D45.RED, D46.RED, D47.RED, D48.RED, D49.RED, D5.RED, D50.RED, D51.RED, D52.RED, D53.RED, D54.RED, D55.RED, D56.RED, D57.RED, D58.RED, D59.RED, D6.RED, D60.RED, D61.RED, D62.RED, D63.RED, D64.RED, D7.RED, D8.RED, D9.RED
- new net N$10: D2.C, IC1G$1.Q6
- new net N$11: D1.C, IC1G$1.Q7
- new net N$12: IC1G$1.DO, IC2G$1.DI
- new net N$13: IC1G$1.SCK, IC2G$1.SCK, IC3G$1.SCK, IC4G$1.SCK, IC5G$1.SCK, IC6G$1.SCK, IC7G$1.SCK, IC8G$1.SCK
- new net N$14: IC1G$1.RCK, IC2G$1.RCK, IC3G$1.RCK, IC4G$1.RCK, IC5G$1.RCK, IC6G$1.RCK, IC7G$1.RCK, IC8G$1.RCK
- new net N$15: D16.C, IC2G$1.Q0
- new net N$16: D15.C, IC2G$1.Q1
- new net N$17: D14.C, IC2G$1.Q2
- new net N$18: D13.C, IC2G$1.Q3
- new net N$19: D12.C, IC2G$1.Q4
- new net N$2: D1.BLU, D10.BLU, D11.BLU, D12.BLU, D13.BLU, D14.BLU, D15.BLU, D16.BLU, D17.BLU, D18.BLU, D19.BLU, D2.BLU, D20.BLU, D21.BLU, D22.BLU, D23.BLU, D24.BLU, D25.BLU, D26.BLU, D27.BLU, D28.BLU, D29.BLU, D3.BLU, D30.BLU, D31.BLU, D32.BLU, D33.BLU, D34.BLU, D35.BLU, D36.BLU, D37.BLU, D38.BLU, D39.BLU, D4.BLU, D40.BLU, D41.BLU, D42.BLU, D43.BLU, D44.BLU, D45.BLU, D46.BLU, D47.BLU, D48.BLU, D49.BLU, D5.BLU, D50.BLU, D51.BLU, D52.BLU, D53.BLU, D54.BLU, D55.BLU, D56.BLU, D57.BLU, D58.BLU, D59.BLU, D6.BLU, D60.BLU, D61.BLU, D62.BLU, D63.BLU, D64.BLU, D7.BLU, D8.BLU, D9.BLU
- new net N$20: D11.C, IC2G$1.Q5
- new net N$21: D10.C, IC2G$1.Q6
- new net N$22: D9.C, IC2G$1.Q7
- new net N$23: D24.C, IC3G$1.Q0
- new net N$24: D23.C, IC3G$1.Q1
- new net N$25: D22.C, IC3G$1.Q2
- new net N$26: D21.C, IC3G$1.Q3
- new net N$27: D20.C, IC3G$1.Q4
- new net N$28: D19.C, IC3G$1.Q5
- new net N$29: D18.C, IC3G$1.Q6
- new net N$3: D1.GRN, D10.GRN, D11.GRN, D12.GRN, D13.GRN, D14.GRN, D15.GRN, D16.GRN, D17.GRN, D18.GRN, D19.GRN, D2.GRN, D20.GRN, D21.GRN, D22.GRN, D23.GRN, D24.GRN, D25.GRN, D26.GRN, D27.GRN, D28.GRN, D29.GRN, D3.GRN, D30.GRN, D31.GRN, D32.GRN, D33.GRN, D34.GRN, D35.GRN, D36.GRN, D37.GRN, D38.GRN, D39.GRN, D4.GRN, D40.GRN, D41.GRN, D42.GRN, D43.GRN, D44.GRN, D45.GRN, D46.GRN, D47.GRN, D48.GRN, D49.GRN, D5.GRN, D50.GRN, D51.GRN, D52.GRN, D53.GRN, D54.GRN, D55.GRN, D56.GRN, D57.GRN, D58.GRN, D59.GRN, D6.GRN, D60.GRN, D61.GRN, D62.GRN, D63.GRN, D64.GRN, D7.GRN, D8.GRN, D9.GRN
- new net N$30: D17.C, IC3G$1.Q7
- new net N$34: IC2G$1.DO, IC3G$1.DI
- new net N$37: D32.C, IC4G$1.Q0
- new net N$38: D31.C, IC4G$1.Q1
- new net N$39: D30.C, IC4G$1.Q2
- new net N$4: D8.C, IC1G$1.Q0
- new net N$40: D29.C, IC4G$1.Q3
- new net N$41: D28.C, IC4G$1.Q4
- new net N$42: D27.C, IC4G$1.Q5
- new net N$43: D26.C, IC4G$1.Q6
- new net N$44: D25.C, IC4G$1.Q7
- new net N$48: IC3G$1.DO, IC4G$1.DI
- new net N$5: D7.C, IC1G$1.Q1
- new net N$51: D40.C, IC5G$1.Q0
- new net N$52: D39.C, IC5G$1.Q1
- new net N$53: D38.C, IC5G$1.Q2
- new net N$54: D37.C, IC5G$1.Q3
- new net N$55: D36.C, IC5G$1.Q4
- new net N$56: D35.C, IC5G$1.Q5
- new net N$57: D34.C, IC5G$1.Q6
- new net N$58: D33.C, IC5G$1.Q7
- new net N$59: IC4G$1.DO, IC5G$1.DI
- new net N$6: D6.C, IC1G$1.Q2
- new net N$65: D48.C, IC6G$1.Q0
- new net N$66: D47.C, IC6G$1.Q1
- new net N$67: D46.C, IC6G$1.Q2
- new net N$68: D45.C, IC6G$1.Q3
- new net N$69: D44.C, IC6G$1.Q4
- new net N$7: D5.C, IC1G$1.Q3
- new net N$70: D43.C, IC6G$1.Q5
- new net N$71: D42.C, IC6G$1.Q6
- new net N$72: D41.C, IC6G$1.Q7
- new net N$73: IC5G$1.DO, IC6G$1.DI
- new net N$74: D56.C, IC7G$1.Q0
- new net N$75: D55.C, IC7G$1.Q1
- new net N$76: D54.C, IC7G$1.Q2
- new net N$77: D53.C, IC7G$1.Q3
- new net N$78: D52.C, IC7G$1.Q4
- new net N$79: D51.C, IC7G$1.Q5
- new net N$8: D4.C, IC1G$1.Q4
- new net N$80: D50.C, IC7G$1.Q6
- new net N$81: D49.C, IC7G$1.Q7
- new net N$82: IC6G$1.DO, IC7G$1.DI
- new net N$83: D64.C, IC8G$1.Q0
- new net N$84: D63.C, IC8G$1.Q1
- new net N$85: D62.C, IC8G$1.Q2
- new net N$86: D61.C, IC8G$1.Q3
- new net N$87: D60.C, IC8G$1.Q4
- new net N$88: D59.C, IC8G$1.Q5
- new net N$89: D58.C, IC8G$1.Q6
- new net N$9: D3.C, IC1G$1.Q5
- new net N$90: D57.C, IC8G$1.Q7
- new net N$91: IC7G$1.DO, IC8G$1.DI
- new net VCC: C1.1, C2.1, C3.1, C4.1, C5.1, C6.1, C7.1, C8.1, IC1G$1.SCLR, IC2G$1.SCLR, IC3G$1.SCLR, IC4G$1.SCLR, IC5G$1.SCLR, IC6G$1.SCLR, IC7G$1.SCLR, IC8G$1.SCLR

Commit message: 2nd layer
Parts:
- added D100, D101, D102, D103, D104, D105, D106, D107, D108, D109, D110, D111, D112, D113, D114, D115, D116, D117, D118, D119, D120, D121, D122, D123, D124, D125, D126, D127, D128, D65, D66, D67, D68, D69, D70, D71, D72, D73, D74, D75, D76, D77, D78, D79, D80, D81, D82, D83, D84, D85, D86, D87, D88, D89, D90, D91, D92, D93, D94, D95, D96, D97, D98, D99: CLEAR, SparkFun-LED:LED-RGB-CCCLEAR
Connections:
- new net N$93: D100.GRN, D101.GRN, D102.GRN, D103.GRN, D104.GRN, D105.GRN, D106.GRN, D107.GRN, D108.GRN, D109.GRN, D110.GRN, D111.GRN, D112.GRN, D113.GRN, D114.GRN, D115.GRN, D116.GRN, D117.GRN, D118.GRN, D119.GRN, D120.GRN, D121.GRN, D122.GRN, D123.GRN, D124.GRN, D125.GRN, D126.GRN, D127.GRN, D128.GRN, D65.GRN, D66.GRN, D67.GRN, D68.GRN, D69.GRN, D70.GRN, D71.GRN, D72.GRN, D73.GRN, D74.GRN, D75.GRN, D76.GRN, D77.GRN, D78.GRN, D79.GRN, D80.GRN, D81.GRN, D82.GRN, D83.GRN, D84.GRN, D85.GRN, D86.GRN, D87.GRN, D88.GRN, D89.GRN, D90.GRN, D91.GRN, D92.GRN, D93.GRN, D94.GRN, D95.GRN, D96.GRN, D97.GRN, D98.GRN, D99.GRN
- new net N$94: D100.BLU, D101.BLU, D102.BLU, D103.BLU, D104.BLU, D105.BLU, D106.BLU, D107.BLU, D108.BLU, D109.BLU, D110.BLU, D111.BLU, D112.BLU, D113.BLU, D114.BLU, D115.BLU, D116.BLU, D117.BLU, D118.BLU, D119.BLU, D120.BLU, D121.BLU, D122.BLU, D123.BLU, D124.BLU, D125.BLU, D126.BLU, D127.BLU, D128.BLU, D65.BLU, D66.BLU, D67.BLU, D68.BLU, D69.BLU, D70.BLU, D71.BLU, D72.BLU, D73.BLU, D74.BLU, D75.BLU, D76.BLU, D77.BLU, D78.BLU, D79.BLU, D80.BLU, D81.BLU, D82.BLU, D83.BLU, D84.BLU, D85.BLU, D86.BLU, D87.BLU, D88.BLU, D89.BLU, D90.BLU, D91.BLU, D92.BLU, D93.BLU, D94.BLU, D95.BLU, D96.BLU, D97.BLU, D98.BLU, D99.BLU
- new net N$95: D100.RED, D101.RED, D102.RED, D103.RED, D104.RED, D105.RED, D106.RED, D107.RED, D108.RED, D109.RED, D110.RED, D111.RED, D112.RED, D113.RED, D114.RED, D115.RED, D116.RED, D117.RED, D118.RED, D119.RED, D120.RED, D121.RED, D122.RED, D123.RED, D124.RED, D125.RED, D126.RED, D127.RED, D128.RED, D65.RED, D66.RED, D67.RED, D68.RED, D69.RED, D70.RED, D71.RED, D72.RED, D73.RED, D74.RED, D75.RED, D76.RED, D77.RED, D78.RED, D79.RED, D80.RED, D81.RED, D82.RED, D83.RED, D84.RED, D85.RED, D86.RED, D87.RED, D88.RED, D89.RED, D90.RED, D91.RED, D92.RED, D93.RED, D94.RED, D95.RED, D96.RED, D97.RED, D98.RED, D99.RED
- net N$10: now also D66.C
- net N$11: now also D65.C
- net N$15: now also D80.C
- net N$16: now also D79.C
- net N$17: now also D78.C
- net N$18: now also D77.C
- net N$19: now also D76.C
- net N$20: now also D75.C
- net N$21: now also D74.C
- net N$22: now also D73.C
- net N$23: now also D88.C
- net N$24: now also D87.C
- net N$25: now also D86.C
- net N$26: now also D85.C
- net N$27: now also D84.C
- net N$28: now also D83.C
- net N$29: now also D82.C
- net N$30: now also D81.C
- net N$37: now also D96.C
- net N$38: now also D95.C
- net N$39: now also D94.C
- net N$4: now also D72.C
- net N$40: now also D93.C
- net N$41: now also D92.C
- net N$42: now also D91.C
- net N$43: now also D90.C
- net N$44: now also D89.C
- net N$5: now also D71.C
- net N$51: now also D104.C
- net N$52: now also D103.C
- net N$53: now also D102.C
- net N$54: now also D101.C
- net N$55: now also D100.C
- net N$56: now also D99.C
- net N$57: now also D98.C
- net N$58: now also D97.C
- net N$6: now also D70.C
- net N$65: now also D112.C
- net N$66: now also D111.C
- net N$67: now also D110.C
- net N$68: now also D109.C
- net N$69: now also D108.C
- net N$7: now also D69.C
- net N$70: now also D107.C
- net N$71: now also D106.C
- net N$72: now also D105.C
- net N$74: now also D120.C
- net N$75: now also D119.C
- net N$76: now also D118.C
- net N$77: now also D117.C
- net N$78: now also D116.C
- net N$79: now also D115.C
- net N$8: now also D68.C
- net N$80: now also D114.C
- net N$81: now also D113.C
- net N$83: now also D128.C
- net N$84: now also D127.C
- net N$85: now also D126.C
- net N$86: now also D125.C
- net N$87: now also D124.C
- net N$88: now also D123.C
- net N$89: now also D122.C
- net N$9: now also D67.C
- net N$90: now also D121.C

Commit message: 3rd layer
Parts:
- added D129, D130, D131, D132, D133, D134, D135, D136, D137, D138, D139, D140, D141, D142, D143, D144, D145, D146, D147, D148, D149, D150, D151, D152, D153, D154, D155, D156, D157, D158, D159, D160, D161, D162, D163, D164, D165, D166, D167, D168, D169, D170, D171, D172, D173, D174, D175, D176, D177, D178, D179, D180, D181, D182, D183, D184, D185, D186, D187, D188, D189, D190, D191, D192: CLEAR, SparkFun-LED:LED-RGB-CCCLEAR
Connections:
- new net N$92: D129.GRN, D130.GRN, D131.GRN, D132.GRN, D133.GRN, D134.GRN, D135.GRN, D136.GRN, D137.GRN, D138.GRN, D139.GRN, D140.GRN, D141.GRN, D142.GRN, D143.GRN, D144.GRN, D145.GRN, D146.GRN, D147.GRN, D148.GRN, D149.GRN, D150.GRN, D151.GRN, D152.GRN, D153.GRN, D154.GRN, D155.GRN, D156.GRN, D157.GRN, D158.GRN, D159.GRN, D160.GRN, D161.GRN, D162.GRN, D163.GRN, D164.GRN, D165.GRN, D166.GRN, D167.GRN, D168.GRN, D169.GRN, D170.GRN, D171.GRN, D172.GRN, D173.GRN, D174.GRN, D175.GRN, D176.GRN, D177.GRN, D178.GRN, D179.GRN, D180.GRN, D181.GRN, D182.GRN, D183.GRN, D184.GRN, D185.GRN, D186.GRN, D187.GRN, D188.GRN, D189.GRN, D190.GRN, D191.GRN, D192.GRN
- new net N$96: D129.BLU, D130.BLU, D131.BLU, D132.BLU, D133.BLU, D134.BLU, D135.BLU, D136.BLU, D137.BLU, D138.BLU, D139.BLU, D140.BLU, D141.BLU, D142.BLU, D143.BLU, D144.BLU, D145.BLU, D146.BLU, D147.BLU, D148.BLU, D149.BLU, D150.BLU, D151.BLU, D152.BLU, D153.BLU, D154.BLU, D155.BLU, D156.BLU, D157.BLU, D158.BLU, D159.BLU, D160.BLU, D161.BLU, D162.BLU, D163.BLU, D164.BLU, D165.BLU, D166.BLU, D167.BLU, D168.BLU, D169.BLU, D170.BLU, D171.BLU, D172.BLU, D173.BLU, D174.BLU, D175.BLU, D176.BLU, D177.BLU, D178.BLU, D179.BLU, D180.BLU, D181.BLU, D182.BLU, D183.BLU, D184.BLU, D185.BLU, D186.BLU, D187.BLU, D188.BLU, D189.BLU, D190.BLU, D191.BLU, D192.BLU
- new net N$97: D129.RED, D130.RED, D131.RED, D132.RED, D133.RED, D134.RED, D135.RED, D136.RED, D137.RED, D138.RED, D139.RED, D140.RED, D141.RED, D142.RED, D143.RED, D144.RED, D145.RED, D146.RED, D147.RED, D148.RED, D149.RED, D150.RED, D151.RED, D152.RED, D153.RED, D154.RED, D155.RED, D156.RED, D157.RED, D158.RED, D159.RED, D160.RED, D161.RED, D162.RED, D163.RED, D164.RED, D165.RED, D166.RED, D167.RED, D168.RED, D169.RED, D170.RED, D171.RED, D172.RED, D173.RED, D174.RED, D175.RED, D176.RED, D177.RED, D178.RED, D179.RED, D180.RED, D181.RED, D182.RED, D183.RED, D184.RED, D185.RED, D186.RED, D187.RED, D188.RED, D189.RED, D190.RED, D191.RED, D192.RED
- net N$10: now also D130.C
- net N$11: now also D129.C
- net N$15: now also D144.C
- net N$16: now also D143.C
- net N$17: now also D142.C
- net N$18: now also D141.C
- net N$19: now also D140.C
- net N$20: now also D139.C
- net N$21: now also D138.C
- net N$22: now also D137.C
- net N$23: now also D152.C
- net N$24: now also D151.C
- net N$25: now also D150.C
- net N$26: now also D149.C
- net N$27: now also D148.C
- net N$28: now also D147.C
- net N$29: now also D146.C
- net N$30: now also D145.C
- net N$37: now also D160.C
- net N$38: now also D159.C
- net N$39: now also D158.C
- net N$4: now also D136.C
- net N$40: now also D157.C
- net N$41: now also D156.C
- net N$42: now also D155.C
- net N$43: now also D154.C
- net N$44: now also D153.C
- net N$5: now also D135.C
- net N$51: now also D168.C
- net N$52: now also D167.C
- net N$53: now also D166.C
- net N$54: now also D165.C
- net N$55: now also D164.C
- net N$56: now also D163.C
- net N$57: now also D162.C
- net N$58: now also D161.C
- net N$6: now also D134.C
- net N$65: now also D176.C
- net N$66: now also D175.C
- net N$67: now also D174.C
- net N$68: now also D173.C
- net N$69: now also D172.C
- net N$7: now also D133.C
- net N$70: now also D171.C
- net N$71: now also D170.C
- net N$72: now also D169.C
- net N$74: now also D184.C
- net N$75: now also D183.C
- net N$76: now also D182.C
- net N$77: now also D181.C
- net N$78: now also D180.C
- net N$79: now also D179.C
- net N$8: now also D132.C
- net N$80: now also D178.C
- net N$81: now also D177.C
- net N$83: now also D192.C
- net N$84: now also D191.C
- net N$85: now also D190.C
- net N$86: now also D189.C
- net N$87: now also D188.C
- net N$88: now also D187.C
- net N$89: now also D186.C
- net N$9: now also D131.C
- net N$90: now also D185.C

Commit message: 4th and 5th layer
Parts:
- added D193, D194, D195, D196, D197, D198, D199, D200, D201, D202, D203, D204, D205, D206, D207, D208, D209, D210, D211, D212, D213, D214, D215, D216, D217, D218, D219, D220, D221, D222, D223, D224, D225, D226, D227, D228, D229, D230, D231, D232, D233, D234, D235, D236, D237, D238, D239, D240, D241, D242, D243, D244, D245, D246, D247, D248, D249, D250, D251, D252, D253, D254, D255, D256, D257, D258, D259, D260, D261, D262, D263, D264, D265, D266, D267, D268, D269, D270, D271, D272, D273, D274, D275, D276, D277, D278, D279, D280, D281, D282, D283, D284, D285, D286, D287, D288, D289, D290, D291, D292, D293, D294, D295, D296, D297, D298, D299, D300, D301, D302, D303, D304, D305, D306, D307, D308, D309, D310, D311, D312, D313, D314, D315, D316, D317, D318, D319, D320: CLEAR, SparkFun-LED:LED-RGB-CCCLEAR
Connections:
- removed net N$86: D125.C, D189.C, D61.C, IC8G$1.Q3
- removed net N$87: D124.C, D188.C, D60.C, IC8G$1.Q4
- removed net N$88: D123.C, D187.C, D59.C, IC8G$1.Q5
- removed net N$89: D122.C, D186.C, D58.C, IC8G$1.Q6
- removed net N$90: D121.C, D185.C, D57.C, IC8G$1.Q7
- new net N$100: D193.RED, D194.RED, D195.RED, D196.RED, D197.RED, D198.RED, D199.RED, D200.RED, D201.RED, D202.RED, D203.RED, D204.RED, D205.RED, D206.RED, D207.RED, D208.RED, D209.RED, D210.RED, D211.RED, D212.RED, D213.RED, D214.RED, D215.RED, D216.RED, D217.RED, D218.RED, D219.RED, D220.RED, D221.RED, D222.RED, D223.RED, D224.RED, D225.RED, D226.RED, D227.RED, D228.RED, D229.RED, D230.RED, D231.RED, D232.RED, D233.RED, D234.RED, D235.RED, D236.RED, D237.RED, D238.RED, D239.RED, D240.RED, D241.RED, D242.RED, D243.RED, D244.RED, D245.RED, D246.RED, D247.RED, D248.RED, D249.RED, D250.RED, D251.RED, D252.RED, D253.RED, D254.RED, D255.RED, D256.RED
- new net N$150: D257.GRN, D258.GRN, D259.GRN, D260.GRN, D261.GRN, D262.GRN, D263.GRN, D264.GRN, D265.GRN, D266.GRN, D267.GRN, D268.GRN, D269.GRN, D270.GRN, D271.GRN, D272.GRN, D273.GRN, D274.GRN, D275.GRN, D276.GRN, D277.GRN, D278.GRN, D279.GRN, D280.GRN, D281.GRN, D282.GRN, D283.GRN, D284.GRN, D285.GRN, D286.GRN, D287.GRN, D288.GRN, D289.GRN, D290.GRN, D291.GRN, D292.GRN, D293.GRN, D294.GRN, D295.GRN, D296.GRN, D297.GRN, D298.GRN, D299.GRN, D300.GRN, D301.GRN, D302.GRN, D303.GRN, D304.GRN, D305.GRN, D306.GRN, D307.GRN, D308.GRN, D309.GRN, D310.GRN, D311.GRN, D312.GRN, D313.GRN, D314.GRN, D315.GRN, D316.GRN, D317.GRN, D318.GRN, D319.GRN, D320.GRN
- new net N$151: D257.BLU, D258.BLU, D259.BLU, D260.BLU, D261.BLU, D262.BLU, D263.BLU, D264.BLU, D265.BLU, D266.BLU, D267.BLU, D268.BLU, D269.BLU, D270.BLU, D271.BLU, D272.BLU, D273.BLU, D274.BLU, D275.BLU, D276.BLU, D277.BLU, D278.BLU, D279.BLU, D280.BLU, D281.BLU, D282.BLU, D283.BLU, D284.BLU, D285.BLU, D286.BLU, D287.BLU, D288.BLU, D289.BLU, D290.BLU, D291.BLU, D292.BLU, D293.BLU, D294.BLU, D295.BLU, D296.BLU, D297.BLU, D298.BLU, D299.BLU, D300.BLU, D301.BLU, D302.BLU, D303.BLU, D304.BLU, D305.BLU, D306.BLU, D307.BLU, D308.BLU, D309.BLU, D310.BLU, D311.BLU, D312.BLU, D313.BLU, D314.BLU, D315.BLU, D316.BLU, D317.BLU, D318.BLU, D319.BLU, D320.BLU
- new net N$152: D257.RED, D258.RED, D259.RED, D260.RED, D261.RED, D262.RED, D263.RED, D264.RED, D265.RED, D266.RED, D267.RED, D268.RED, D269.RED, D270.RED, D271.RED, D272.RED, D273.RED, D274.RED, D275.RED, D276.RED, D277.RED, D278.RED, D279.RED, D280.RED, D281.RED, D282.RED, D283.RED, D284.RED, D285.RED, D286.RED, D287.RED, D288.RED, D289.RED, D290.RED, D291.RED, D292.RED, D293.RED, D294.RED, D295.RED, D296.RED, D297.RED, D298.RED, D299.RED, D300.RED, D301.RED, D302.RED, D303.RED, D304.RED, D305.RED, D306.RED, D307.RED, D308.RED, D309.RED, D310.RED, D311.RED, D312.RED, D313.RED, D314.RED, D315.RED, D316.RED, D317.RED, D318.RED, D319.RED, D320.RED
- new net N$60: D125.C, D189.C, D253.C, D317.C, D61.C, IC8G$1.Q3
- new net N$61: D124.C, D188.C, D252.C, D316.C, D60.C, IC8G$1.Q4
- new net N$62: D123.C, D187.C, D251.C, D315.C, D59.C, IC8G$1.Q5
- new net N$63: D122.C, D186.C, D250.C, D314.C, D58.C, IC8G$1.Q6
- new net N$64: D121.C, D185.C, D249.C, D313.C, D57.C, IC8G$1.Q7
- new net N$98: D193.GRN, D194.GRN, D195.GRN, D196.GRN, D197.GRN, D198.GRN, D199.GRN, D200.GRN, D201.GRN, D202.GRN, D203.GRN, D204.GRN, D205.GRN, D206.GRN, D207.GRN, D208.GRN, D209.GRN, D210.GRN, D211.GRN, D212.GRN, D213.GRN, D214.GRN, D215.GRN, D216.GRN, D217.GRN, D218.GRN, D219.GRN, D220.GRN, D221.GRN, D222.GRN, D223.GRN, D224.GRN, D225.GRN, D226.GRN, D227.GRN, D228.GRN, D229.GRN, D230.GRN, D231.GRN, D232.GRN, D233.GRN, D234.GRN, D235.GRN, D236.GRN, D237.GRN, D238.GRN, D239.GRN, D240.GRN, D241.GRN, D242.GRN, D243.GRN, D244.GRN, D245.GRN, D246.GRN, D247.GRN, D248.GRN, D249.GRN, D250.GRN, D251.GRN, D252.GRN, D253.GRN, D254.GRN, D255.GRN, D256.GRN
- new net N$99: D193.BLU, D194.BLU, D195.BLU, D196.BLU, D197.BLU, D198.BLU, D199.BLU, D200.BLU, D201.BLU, D202.BLU, D203.BLU, D204.BLU, D205.BLU, D206.BLU, D207.BLU, D208.BLU, D209.BLU, D210.BLU, D211.BLU, D212.BLU, D213.BLU, D214.BLU, D215.BLU, D216.BLU, D217.BLU, D218.BLU, D219.BLU, D220.BLU, D221.BLU, D222.BLU, D223.BLU, D224.BLU, D225.BLU, D226.BLU, D227.BLU, D228.BLU, D229.BLU, D230.BLU, D231.BLU, D232.BLU, D233.BLU, D234.BLU, D235.BLU, D236.BLU, D237.BLU, D238.BLU, D239.BLU, D240.BLU, D241.BLU, D242.BLU, D243.BLU, D244.BLU, D245.BLU, D246.BLU, D247.BLU, D248.BLU, D249.BLU, D250.BLU, D251.BLU, D252.BLU, D253.BLU, D254.BLU, D255.BLU, D256.BLU
- net N$10: now also D194.C, D258.C
- net N$11: now also D193.C, D257.C
- net N$15: now also D208.C, D272.C
- net N$16: now also D207.C, D271.C
- net N$17: now also D206.C, D270.C
- net N$18: now also D205.C, D269.C
- net N$19: now also D204.C, D268.C
- net N$20: now also D203.C, D267.C
- net N$21: now also D202.C, D266.C
- net N$22: now also D201.C, D265.C
- net N$23: now also D216.C, D280.C
- net N$24: now also D215.C, D279.C
- net N$25: now also D214.C, D278.C
- net N$26: now also D213.C, D277.C
- net N$27: now also D212.C, D276.C
- net N$28: now also D211.C, D275.C
- net N$29: now also D210.C, D274.C
- net N$30: now also D209.C, D273.C
- net N$37: now also D224.C, D288.C
- net N$38: now also D223.C, D287.C
- net N$39: now also D222.C, D286.C
- net N$4: now also D200.C, D264.C
- net N$40: now also D221.C, D285.C
- net N$41: now also D220.C, D284.C
- net N$42: now also D219.C, D283.C
- net N$43: now also D218.C, D282.C
- net N$44: now also D217.C, D281.C
- net N$5: now also D199.C, D263.C
- net N$51: now also D232.C, D296.C
- net N$52: now also D231.C, D295.C
- net N$53: now also D230.C, D294.C
- net N$54: now also D229.C, D293.C
- net N$55: now also D228.C, D292.C
- net N$56: now also D227.C, D291.C
- net N$57: now also D226.C, D290.C
- net N$58: now also D225.C, D289.C
- net N$6: now also D198.C, D262.C
- net N$65: now also D240.C, D304.C
- net N$66: now also D239.C, D303.C
- net N$67: now also D238.C, D302.C
- net N$68: now also D237.C, D301.C
- net N$69: now also D236.C, D300.C
- net N$7: now also D197.C, D261.C
- net N$70: now also D235.C, D299.C
- net N$71: now also D234.C, D298.C
- net N$72: now also D233.C, D297.C
- net N$74: now also D248.C, D312.C
- net N$75: now also D247.C, D311.C
- net N$76: now also D246.C, D310.C
- net N$77: now also D245.C, D309.C
- net N$78: now also D244.C, D308.C
- net N$79: now also D243.C, D307.C
- net N$8: now also D196.C, D260.C
- net N$80: now also D242.C, D306.C
- net N$81: now also D241.C, D305.C
- net N$83: now also D256.C, D320.C
- net N$84: now also D255.C, D319.C
- net N$85: now also D254.C, D318.C
- net N$9: now also D195.C, D259.C

Commit message: 6th 7th and 8th layer
Parts:
- added D321, D322, D323, D324, D325, D326, D327, D328, D329, D330, D331, D332, D333, D334, D335, D336, D337, D338, D339, D340, D341, D342, D343, D344, D345, D346, D347, D348, D349, D350, D351, D352, D353, D354, D355, D356, D357, D358, D359, D360, D361, D362, D363, D364, D365, D366, D367, D368, D369, D370, D371, D372, D373, D374, D375, D376, D377, D378, D379, D380, D381, D382, D383, D384, D385, D386, D387, D388, D389, D390, D391, D392, D393, D394, D395, D396, D397, D398, D399, D400, D401, D402, D403, D404, D405, D406, D407, D408, D409, D410, D411, D412, D413, D414, D415, D416, D417, D418, D419, D420, D421, D422, D423, D424, D425, D426, D427, D428, D429, D430, D431, D432, D433, D434, D435, D436, D437, D438, D439, D440, D441, D442, D443, D444, D445, D446, D447, D448, D449, D450, D451, D452, D453, D454, D455, D456, D457, D458, D459, D460, D461, D462, D463, D464, D465, D466, D467, D468, D469, D470, D471, D472, D473, D474, D475, D476, D477, D478, D479, D480, D481, D482, D483, D484, D485, D486, D487, D488, D489, D490, D491, D492, D493, D494, D495, D496, D497, D498, D499, D500, D501, D502, D503, D504, D505, D506, D507, D508, D509, D510, D511, D512: CLEAR, SparkFun-LED:LED-RGB-CCCLEAR
Connections:
- new net N$145: D321.GRN, D322.GRN, D323.GRN, D324.GRN, D325.GRN, D326.GRN, D327.GRN, D328.GRN, D329.GRN, D330.GRN, D331.GRN, D332.GRN, D333.GRN, D334.GRN, D335.GRN, D336.GRN, D337.GRN, D338.GRN, D339.GRN, D340.GRN, D341.GRN, D342.GRN, D343.GRN, D344.GRN, D345.GRN, D346.GRN, D347.GRN, D348.GRN, D349.GRN, D350.GRN, D351.GRN, D352.GRN, D353.GRN, D354.GRN, D355.GRN, D356.GRN, D357.GRN, D358.GRN, D359.GRN, D360.GRN, D361.GRN, D362.GRN, D363.GRN, D364.GRN, D365.GRN, D366.GRN, D367.GRN, D368.GRN, D369.GRN, D370.GRN, D371.GRN, D372.GRN, D373.GRN, D374.GRN, D375.GRN, D376.GRN, D377.GRN, D378.GRN, D379.GRN, D380.GRN, D381.GRN, D382.GRN, D383.GRN, D384.GRN
- new net N$146: D321.BLU, D322.BLU, D323.BLU, D324.BLU, D325.BLU, D326.BLU, D327.BLU, D328.BLU, D329.BLU, D330.BLU, D331.BLU, D332.BLU, D333.BLU, D334.BLU, D335.BLU, D336.BLU, D337.BLU, D338.BLU, D339.BLU, D340.BLU, D341.BLU, D342.BLU, D343.BLU, D344.BLU, D345.BLU, D346.BLU, D347.BLU, D348.BLU, D349.BLU, D350.BLU, D351.BLU, D352.BLU, D353.BLU, D354.BLU, D355.BLU, D356.BLU, D357.BLU, D358.BLU, D359.BLU, D360.BLU, D361.BLU, D362.BLU, D363.BLU, D364.BLU, D365.BLU, D366.BLU, D367.BLU, D368.BLU, D369.BLU, D370.BLU, D371.BLU, D372.BLU, D373.BLU, D374.BLU, D375.BLU, D376.BLU, D377.BLU, D378.BLU, D379.BLU, D380.BLU, D381.BLU, D382.BLU, D383.BLU, D384.BLU
- new net N$147: D321.RED, D322.RED, D323.RED, D324.RED, D325.RED, D326.RED, D327.RED, D328.RED, D329.RED, D330.RED, D331.RED, D332.RED, D333.RED, D334.RED, D335.RED, D336.RED, D337.RED, D338.RED, D339.RED, D340.RED, D341.RED, D342.RED, D343.RED, D344.RED, D345.RED, D346.RED, D347.RED, D348.RED, D349.RED, D350.RED, D351.RED, D352.RED, D353.RED, D354.RED, D355.RED, D356.RED, D357.RED, D358.RED, D359.RED, D360.RED, D361.RED, D362.RED, D363.RED, D364.RED, D365.RED, D366.RED, D367.RED, D368.RED, D369.RED, D370.RED, D371.RED, D372.RED, D373.RED, D374.RED, D375.RED, D376.RED, D377.RED, D378.RED, D379.RED, D380.RED, D381.RED, D382.RED, D383.RED, D384.RED
- new net N$148: D385.GRN, D386.GRN, D387.GRN, D388.GRN, D389.GRN, D390.GRN, D391.GRN, D392.GRN, D393.GRN, D394.GRN, D395.GRN, D396.GRN, D397.GRN, D398.GRN, D399.GRN, D400.GRN, D401.GRN, D402.GRN, D403.GRN, D404.GRN, D405.GRN, D406.GRN, D407.GRN, D408.GRN, D409.GRN, D410.GRN, D411.GRN, D412.GRN, D413.GRN, D414.GRN, D415.GRN, D416.GRN, D417.GRN, D418.GRN, D419.GRN, D420.GRN, D421.GRN, D422.GRN, D423.GRN, D424.GRN, D425.GRN, D426.GRN, D427.GRN, D428.GRN, D429.GRN, D430.GRN, D431.GRN, D432.GRN, D433.GRN, D434.GRN, D435.GRN, D436.GRN, D437.GRN, D438.GRN, D439.GRN, D440.GRN, D441.GRN, D442.GRN, D443.GRN, D444.GRN, D445.GRN, D446.GRN, D447.GRN, D448.GRN
- new net N$149: D385.BLU, D386.BLU, D387.BLU, D388.BLU, D389.BLU, D390.BLU, D391.BLU, D392.BLU, D393.BLU, D394.BLU, D395.BLU, D396.BLU, D397.BLU, D398.BLU, D399.BLU, D400.BLU, D401.BLU, D402.BLU, D403.BLU, D404.BLU, D405.BLU, D406.BLU, D407.BLU, D408.BLU, D409.BLU, D410.BLU, D411.BLU, D412.BLU, D413.BLU, D414.BLU, D415.BLU, D416.BLU, D417.BLU, D418.BLU, D419.BLU, D420.BLU, D421.BLU, D422.BLU, D423.BLU, D424.BLU, D425.BLU, D426.BLU, D427.BLU, D428.BLU, D429.BLU, D430.BLU, D431.BLU, D432.BLU, D433.BLU, D434.BLU, D435.BLU, D436.BLU, D437.BLU, D438.BLU, D439.BLU, D440.BLU, D441.BLU, D442.BLU, D443.BLU, D444.BLU, D445.BLU, D446.BLU, D447.BLU, D448.BLU
- new net N$153: D385.RED, D386.RED, D387.RED, D388.RED, D389.RED, D390.RED, D391.RED, D392.RED, D393.RED, D394.RED, D395.RED, D396.RED, D397.RED, D398.RED, D399.RED, D400.RED, D401.RED, D402.RED, D403.RED, D404.RED, D405.RED, D406.RED, D407.RED, D408.RED, D409.RED, D410.RED, D411.RED, D412.RED, D413.RED, D414.RED, D415.RED, D416.RED, D417.RED, D418.RED, D419.RED, D420.RED, D421.RED, D422.RED, D423.RED, D424.RED, D425.RED, D426.RED, D427.RED, D428.RED, D429.RED, D430.RED, D431.RED, D432.RED, D433.RED, D434.RED, D435.RED, D436.RED, D437.RED, D438.RED, D439.RED, D440.RED, D441.RED, D442.RED, D443.RED, D444.RED, D445.RED, D446.RED, D447.RED, D448.RED
- new net N$154: D449.GRN, D450.GRN, D451.GRN, D452.GRN, D453.GRN, D454.GRN, D455.GRN, D456.GRN, D457.GRN, D458.GRN, D459.GRN, D460.GRN, D461.GRN, D462.GRN, D463.GRN, D464.GRN, D465.GRN, D466.GRN, D467.GRN, D468.GRN, D469.GRN, D470.GRN, D471.GRN, D472.GRN, D473.GRN, D474.GRN, D475.GRN, D476.GRN, D477.GRN, D478.GRN, D479.GRN, D480.GRN, D481.GRN, D482.GRN, D483.GRN, D484.GRN, D485.GRN, D486.GRN, D487.GRN, D488.GRN, D489.GRN, D490.GRN, D491.GRN, D492.GRN, D493.GRN, D494.GRN, D495.GRN, D496.GRN, D497.GRN, D498.GRN, D499.GRN, D500.GRN, D501.GRN, D502.GRN, D503.GRN, D504.GRN, D505.GRN, D506.GRN, D507.GRN, D508.GRN, D509.GRN, D510.GRN, D511.GRN, D512.GRN
- new net N$155: D449.BLU, D450.BLU, D451.BLU, D452.BLU, D453.BLU, D454.BLU, D455.BLU, D456.BLU, D457.BLU, D458.BLU, D459.BLU, D460.BLU, D461.BLU, D462.BLU, D463.BLU, D464.BLU, D465.BLU, D466.BLU, D467.BLU, D468.BLU, D469.BLU, D470.BLU, D471.BLU, D472.BLU, D473.BLU, D474.BLU, D475.BLU, D476.BLU, D477.BLU, D478.BLU, D479.BLU, D480.BLU, D481.BLU, D482.BLU, D483.BLU, D484.BLU, D485.BLU, D486.BLU, D487.BLU, D488.BLU, D489.BLU, D490.BLU, D491.BLU, D492.BLU, D493.BLU, D494.BLU, D495.BLU, D496.BLU, D497.BLU, D498.BLU, D499.BLU, D500.BLU, D501.BLU, D502.BLU, D503.BLU, D504.BLU, D505.BLU, D506.BLU, D507.BLU, D508.BLU, D509.BLU, D510.BLU, D511.BLU, D512.BLU
- new net N$156: D449.RED, D450.RED, D451.RED, D452.RED, D453.RED, D454.RED, D455.RED, D456.RED, D457.RED, D458.RED, D459.RED, D460.RED, D461.RED, D462.RED, D463.RED, D464.RED, D465.RED, D466.RED, D467.RED, D468.RED, D469.RED, D470.RED, D471.RED, D472.RED, D473.RED, D474.RED, D475.RED, D476.RED, D477.RED, D478.RED, D479.RED, D480.RED, D481.RED, D482.RED, D483.RED, D484.RED, D485.RED, D486.RED, D487.RED, D488.RED, D489.RED, D490.RED, D491.RED, D492.RED, D493.RED, D494.RED, D495.RED, D496.RED, D497.RED, D498.RED, D499.RED, D500.RED, D501.RED, D502.RED, D503.RED, D504.RED, D505.RED, D506.RED, D507.RED, D508.RED, D509.RED, D510.RED, D511.RED, D512.RED
- net N$10: now also D322.C, D386.C, D450.C
- net N$11: now also D321.C, D385.C, D449.C
- net N$15: now also D336.C, D400.C, D464.C
- net N$16: now also D335.C, D399.C, D463.C
- net N$17: now also D334.C, D398.C, D462.C
- net N$18: now also D333.C, D397.C, D461.C
- net N$19: now also D332.C, D396.C, D460.C
- net N$20: now also D331.C, D395.C, D459.C
- net N$21: now also D330.C, D394.C, D458.C
- net N$22: now also D329.C, D393.C, D457.C
- net N$23: now also D344.C, D408.C, D472.C
- net N$24: now also D343.C, D407.C, D471.C
- net N$25: now also D342.C, D406.C, D470.C
- net N$26: now also D341.C, D405.C, D469.C
- net N$27: now also D340.C, D404.C, D468.C
- net N$28: now also D339.C, D403.C, D467.C
- net N$29: now also D338.C, D402.C, D466.C
- net N$30: now also D337.C, D401.C, D465.C
- net N$37: now also D352.C, D416.C, D480.C
- net N$38: now also D351.C, D415.C, D479.C
- net N$39: now also D350.C, D414.C, D478.C
- net N$4: now also D328.C, D392.C, D456.C
- net N$40: now also D349.C, D413.C, D477.C
- net N$41: now also D348.C, D412.C, D476.C
- net N$42: now also D347.C, D411.C, D475.C
- net N$43: now also D346.C, D410.C, D474.C
- net N$44: now also D345.C, D409.C, D473.C
- net N$5: now also D327.C, D391.C, D455.C
- net N$51: now also D360.C, D424.C, D488.C
- net N$52: now also D359.C, D423.C, D487.C
- net N$53: now also D358.C, D422.C, D486.C
- net N$54: now also D357.C, D421.C, D485.C
- net N$55: now also D356.C, D420.C, D484.C
- net N$56: now also D355.C, D419.C, D483.C
- net N$57: now also D354.C, D418.C, D482.C
- net N$58: now also D353.C, D417.C, D481.C
- net N$6: now also D326.C, D390.C, D454.C
- net N$60: now also D381.C, D445.C, D509.C
- net N$61: now also D380.C, D444.C, D508.C
- net N$62: now also D379.C, D443.C, D507.C
- net N$63: now also D378.C, D442.C, D506.C
- net N$64: now also D377.C, D441.C, D505.C
- net N$65: now also D368.C, D432.C, D496.C
- net N$66: now also D367.C, D431.C, D495.C
- net N$67: now also D366.C, D430.C, D494.C
- net N$68: now also D365.C, D429.C, D493.C
- net N$69: now also D364.C, D428.C, D492.C
- net N$7: now also D325.C, D389.C, D453.C
- net N$70: now also D363.C, D427.C, D491.C
- net N$71: now also D362.C, D426.C, D490.C
- net N$72: now also D361.C, D425.C, D489.C
- net N$74: now also D376.C, D440.C, D504.C
- net N$75: now also D375.C, D439.C, D503.C
- net N$76: now also D374.C, D438.C, D502.C
- net N$77: now also D373.C, D437.C, D501.C
- net N$78: now also D372.C, D436.C, D500.C
- net N$79: now also D371.C, D435.C, D499.C
- net N$8: now also D324.C, D388.C, D452.C
- net N$80: now also D370.C, D434.C, D498.C
- net N$81: now also D369.C, D433.C, D497.C
- net N$83: now also D384.C, D448.C, D512.C
- net N$84: now also D383.C, D447.C, D511.C
- net N$85: now also D382.C, D446.C, D510.C
- net N$9: now also D323.C, D387.C, D451.C

Commit message: added connections for the level
Parts:
- added C10, C11, C12, C13, C14, C9: 100n, rcl:C-EU050-024X044
- added IC10, IC11, IC9: UDN2981A, uln-udn:UDN2981A
- added IC12, IC13, IC14: 74HC595N, 74xx-eu:74HC595N
Connections:
- removed net N$145: D321.GRN, D322.GRN, D323.GRN, D324.GRN, D325.GRN, D326.GRN, D327.GRN, D328.GRN, D329.GRN, D330.GRN, D331.GRN, D332.GRN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
- removed net N$146: D321.BLU, D322.BLU, D323.BLU, D324.BLU, D325.BLU, D326.BLU, D327.BLU, D328.BLU, D329.BLU, D330.BLU, D331.BLU, D332.BLU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
- removed net N$148: D385.GRN, D386.GRN, D387.GRN, D388.GRN, D389.GRN, D390.GRN, D391.GRN, D392.GRN, D393.GRN, D394.GRN, D395.GRN, D396.GRN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
- removed net N$149: D385.BLU, D386.BLU, D387.BLU, D388.BLU, D389.BLU, D390.BLU, D391.BLU, D392.BLU, D393.BLU, D394.BLU, D395.BLU, D396.BLU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
- removed net N$150: D257.GRN, D258.GRN, D259.GRN, D260.GRN, D261.GRN, D262.GRN, D263.GRN, D264.GRN, D265.GRN, D266.GRN, D267.GRN, D268.GRN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
- removed net N$151: D257.BLU, D258.BLU, D259.BLU, D260.BLU, D261.BLU, D262.BLU, D263.BLU, D264.BLU, D265.BLU, D266.BLU, D267.BLU, D268.BLU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
- removed net N$154: D449.GRN, D450.GRN, D451.GRN, D452.GRN, D453.GRN, D454.GRN, D455.GRN, D456.GRN, D457.GRN, D458.GRN, D459.GRN, D460.GRN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
- removed net N$155: D449.BLU, D450.BLU, D451.BLU, D452.BLU, D453.BLU, D454.BLU, D455.BLU, D456.BLU, D457.BLU, D458.BLU, D459.BLU, D460.BLU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
- new net N$101: IC12A.QF, IC9.I6
- new net N$102: D449.GRN, D450.GRN, D451.GRN, D452.GRN, D453.GRN, D454.GRN, D455.GRN, D456.GRN, D457.GRN, D458.GRN, D459.GRN, D460.GRN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
- new net N$103: D385.GRN, D386.GRN, D387.GRN, D388.GRN, D389.GRN, D390.GRN, D391.GRN, D392.GRN, D393.GRN, D394.GRN, D395.GRN, D396.GRN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
- new net N$104: D321.GRN, D322.GRN, D323.GRN, D324.GRN, D325.GRN, D326.GRN, D327.GRN, D328.GRN, D329.GRN, D330.GRN, D331.GRN, D332.GRN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
- new net N$105: D257.GRN, D258.GRN, D259.GRN, D260.GRN, D261.GRN, D262.GRN, D263.GRN, D264.GRN, D265.GRN, D266.GRN, D267.GRN, D268.GRN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
- new net N$106: IC12A.QG, IC9.I7
- new net N$107: IC12A.QH, IC9.I8
- new net N$108: IC12A.QH*, IC1G$1.DI
- new net N$109: IC11.I3, IC14A.QC
- new net N$110: IC11.I4, IC14A.QD
- new net N$111: IC10.I1, IC13A.QA
- new net N$112: IC10.I2, IC13A.QB
- new net N$113: IC10.I3, IC13A.QC
- new net N$114: IC10.I4, IC13A.QD
- new net N$115: IC10.I5, IC13A.QE
- new net N$116: IC10.I6, IC13A.QF
- new net N$117: IC10.I7, IC13A.QG
- new net N$118: IC10.I8, IC13A.QH
- new net N$119: IC12A.SER, IC13A.QH*
- new net N$120: IC11.I5, IC14A.QE
- new net N$121: IC11.I6, IC14A.QF
- new net N$122: IC11.I7, IC14A.QG
- new net N$123: IC11.I8, IC14A.QH
- new net N$124: IC13A.SER, IC14A.QH*
- new net N$31: IC11.I1, IC14A.QA
- new net N$32: IC11.I2, IC14A.QB
- new net N$46: IC12A.QA, IC9.I1
- new net N$47: IC12A.QB, IC9.I2
- new net N$49: D100.BLU, D101.BLU, D102.BLU, D103.BLU, D104.BLU, D105.BLU, D106.BLU, D107.BLU, D108.BLU, D109.BLU, D110.BLU, D111.BLU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
- new net N$50: D129.BLU, D130.BLU, D131.BLU, D132.BLU, D133.BLU, D134.BLU, D135.BLU, D136.BLU, D137.BLU, D138.BLU, D139.BLU, D140.BLU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
- new net N$86: D193.BLU, D194.BLU, D195.BLU, D196.BLU, D197.BLU, D198.BLU, D199.BLU, D200.BLU, D201.BLU, D202.BLU, D203.BLU, D204.BLU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
- new net N$87: D257.BLU, D258.BLU, D259.BLU, D260.BLU, D261.BLU, D262.BLU, D263.BLU, D264.BLU, D265.BLU, D266.BLU, D267.BLU, D268.BLU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
- new net N$88: D321.BLU, D322.BLU, D323.BLU, D324.BLU, D325.BLU, D326.BLU, D327.BLU, D328.BLU, D329.BLU, D330.BLU, D331.BLU, D332.BLU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
- new net N$89: D385.BLU, D386.BLU, D387.BLU, D388.BLU, D389.BLU, D390.BLU, D391.BLU, D392.BLU, D393.BLU, D394.BLU, D395.BLU, D396.BLU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
- new net N$90: D449.BLU, D450.BLU, D451.BLU, D452.BLU, D453.BLU, D454.BLU, D455.BLU, D456.BLU, D457.BLU, D458.BLU, D459.BLU, D460.BLU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
- net GND: now also C10.2, C11.2, C12.2, C13.2, C14.2, C9.2, IC10.GND, IC11.GND, IC12A.G, IC13A.G, IC14A.G, IC9.GND
- net N$1: now also IC9.O8
- net N$100: now also IC9.O5
- net N$13: now also IC12A.SCK, IC13A.SCK, IC14A.SCK
- net N$14: now also IC12A.RCK, IC13A.RCK, IC14A.RCK
- net N$147: now also IC9.O3
- net N$152: now also IC9.O4
- net N$153: now also IC9.O2
- net N$156: now also IC9.O1
- net N$2: now also IC10.O8
- net N$3: now also IC11.O8
- net N$92: now also IC11.O6
- net N$93: now also IC11.O7
- net N$94: now also IC12A.QC, IC9.I3; no longer D100.BLU, D101.BLU, D102.BLU, D103.BLU, D104.BLU, D105.BLU, D106.BLU, D107.BLU, D108.BLU, D109.BLU, D110.BLU, D111.BLU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
- net N$95: now also IC9.O7
- net N$96: now also IC12A.QD, IC9.I4; no longer D129.BLU, D130.BLU, D131.BLU, D132.BLU, D133.BLU, D134.BLU, D135.BLU, D136.BLU, D137.BLU, D138.BLU, D139.BLU, D140.BLU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
- net N$97: now also IC9.O6
- net N$98: now also IC11.O5
- net N$99: now also IC12A.QE, IC9.I5; no longer D193.BLU, D194.BLU, D195.BLU, D196.BLU, D197.BLU, D198.BLU, D199.BLU, D200.BLU, D201.BLU, D202.BLU, D203.BLU, D204.BLU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
- net VCC: now also C10.1, C11.1, C12.1, C13.1, C14.1, C9.1, IC10.VS, IC11.VS, IC12A.SCL, IC13A.SCL, IC14A.SCL, IC9.VS
