File: cube.sch (EAGLE design)
At the start: 540 parts, among them IC1 TPIC6B595N, IC10 UDN2981A, IC11 UDN2981A, IC12 74HC595N, IC13 74HC595N, IC14 74HC595N, IC2 TPIC6B595N, IC3 TPIC6B595N, IC4 TPIC6B595N, IC5 TPIC6B595N, IC6 TPIC6B595N, IC7 TPIC6B595N, IC8 TPIC6B595N, IC9 UDN2981A

Commit message: added resistors to the leds
Parts:
- added R1, R10, R11, R12, R13, R14, R15, R16, R17, R18, R19, R2, R20, R21, R22, R23, R24, R25, R26, R27, R28, R29, R3, R30, R31, R32, R33, R34, R35, R36, R37, R38, R39, R4, R40, R41, R42, R43, R44, R45, R46, R47, R48, R49, R5, R50, R51, R52, R53, R54, R55, R56, R57, R58, R59, R6, R60, R61, R62, R63, R64, R7, R8, R9: 150R, rcl:R-EU_0207/10
Connections:
- new net N$125: IC1G$1.Q6, R7.1
- new net N$126: IC1G$1.Q7, R8.1
- new net N$127: IC1G$1.Q5, R6.1
- new net N$128: IC1G$1.Q3, R4.1
- new net N$129: IC2G$1.Q7, R16.1
- new net N$130: IC2G$1.Q6, R15.1
- new net N$131: IC2G$1.Q5, R14.1
- new net N$132: IC2G$1.Q4, R13.1
- new net N$133: IC2G$1.Q3, R12.1
- new net N$134: IC2G$1.Q2, R11.1
- new net N$135: IC2G$1.Q1, R10.1
- new net N$136: IC2G$1.Q0, R9.1
- new net N$137: IC3G$1.Q7, R24.1
- new net N$138: IC3G$1.Q6, R23.1
- new net N$139: IC3G$1.Q5, R22.1
- new net N$140: IC3G$1.Q4, R21.1
- new net N$141: IC3G$1.Q3, R20.1
- new net N$142: IC3G$1.Q2, R19.1
- new net N$143: IC3G$1.Q1, R18.1
- new net N$144: IC3G$1.Q0, R17.1
- new net N$145: IC4G$1.Q7, R32.1
- new net N$146: IC4G$1.Q6, R31.1
- new net N$148: IC4G$1.Q5, R30.1
- new net N$149: IC4G$1.Q4, R29.1
- new net N$150: IC4G$1.Q3, R28.1
- new net N$151: IC4G$1.Q2, R27.1
- new net N$154: IC4G$1.Q1, R26.1
- new net N$155: IC4G$1.Q0, R25.1
- new net N$157: IC8G$1.Q7, R64.1
- new net N$158: IC8G$1.Q6, R63.1
- new net N$159: IC8G$1.Q5, R62.1
- new net N$160: IC8G$1.Q4, R61.1
- new net N$161: IC8G$1.Q3, R60.1
- new net N$162: IC8G$1.Q2, R59.1
- new net N$163: IC8G$1.Q1, R58.1
- new net N$164: IC8G$1.Q0, R57.1
- new net N$165: IC7G$1.Q0, R49.1
- new net N$166: IC7G$1.Q1, R50.1
- new net N$167: IC7G$1.Q2, R51.1
- new net N$168: IC7G$1.Q3, R52.1
- new net N$169: IC7G$1.Q4, R53.1
- new net N$170: IC7G$1.Q5, R54.1
- new net N$171: IC7G$1.Q6, R55.1
- new net N$172: IC7G$1.Q7, R56.1
- new net N$173: IC6G$1.Q7, R48.1
- new net N$174: IC6G$1.Q6, R47.1
- new net N$175: IC6G$1.Q5, R46.1
- new net N$176: IC6G$1.Q4, R45.1
- new net N$177: IC6G$1.Q3, R44.1
- new net N$178: IC6G$1.Q2, R43.1
- new net N$179: IC6G$1.Q1, R42.1
- new net N$180: IC6G$1.Q0, R41.1
- new net N$181: IC5G$1.Q0, R33.1
- new net N$182: IC5G$1.Q1, R34.1
- new net N$183: IC5G$1.Q2, R35.1
- new net N$184: IC5G$1.Q3, R36.1
- new net N$185: IC5G$1.Q4, R37.1
- new net N$186: IC5G$1.Q5, R38.1
- new net N$187: IC5G$1.Q6, R39.1
- new net N$188: IC5G$1.Q7, R40.1
- new net N$33: IC1G$1.Q0, R1.1
- new net N$35: IC1G$1.Q1, R2.1
- new net N$36: IC1G$1.Q2, R3.1
- new net N$45: IC1G$1.Q4, R5.1
- net N$10: now also R7.2; no longer IC1G$1.Q6
- net N$11: now also R8.2; no longer IC1G$1.Q7
- net N$15: now also R9.2; no longer IC2G$1.Q0
- net N$16: now also R10.2; no longer IC2G$1.Q1
- net N$17: now also R11.2; no longer IC2G$1.Q2
- net N$18: now also R12.2; no longer IC2G$1.Q3
- net N$19: now also R13.2; no longer IC2G$1.Q4
- net N$20: now also R14.2; no longer IC2G$1.Q5
- net N$21: now also R15.2; no longer IC2G$1.Q6
- net N$22: now also R16.2; no longer IC2G$1.Q7
- net N$23: now also R17.2; no longer IC3G$1.Q0
- net N$24: now also R18.2; no longer IC3G$1.Q1
- net N$25: now also R19.2; no longer IC3G$1.Q2
- net N$26: now also R20.2; no longer IC3G$1.Q3
- net N$27: now also R21.2; no longer IC3G$1.Q4
- net N$28: now also R22.2; no longer IC3G$1.Q5
- net N$29: now also R23.2; no longer IC3G$1.Q6
- net N$30: now also R24.2; no longer IC3G$1.Q7
- net N$37: now also R25.2; no longer IC4G$1.Q0
- net N$38: now also R26.2; no longer IC4G$1.Q1
- net N$39: now also R27.2; no longer IC4G$1.Q2
- net N$4: now also R1.2; no longer IC1G$1.Q0
- net N$40: now also R28.2; no longer IC4G$1.Q3
- net N$41: now also R29.2; no longer IC4G$1.Q4
- net N$42: now also R30.2; no longer IC4G$1.Q5
- net N$43: now also R31.2; no longer IC4G$1.Q6
- net N$44: now also R32.2; no longer IC4G$1.Q7
- net N$5: now also R2.2; no longer IC1G$1.Q1
- net N$51: now also R33.2; no longer IC5G$1.Q0
- net N$52: now also R34.2; no longer IC5G$1.Q1
- net N$53: now also R35.2; no longer IC5G$1.Q2
- net N$54: now also R36.2; no longer IC5G$1.Q3
- net N$55: now also R37.2; no longer IC5G$1.Q4
- net N$56: now also R38.2; no longer IC5G$1.Q5
- net N$57: now also R39.2; no longer IC5G$1.Q6
- net N$58: now also R40.2; no longer IC5G$1.Q7
- net N$6: now also R3.2; no longer IC1G$1.Q2
- net N$60: now also R60.2; no longer IC8G$1.Q3
- net N$61: now also R61.2; no longer IC8G$1.Q4
- net N$62: now also R62.2; no longer IC8G$1.Q5
- net N$63: now also R63.2; no longer IC8G$1.Q6
- net N$64: now also R64.2; no longer IC8G$1.Q7
- net N$65: now also R41.2; no longer IC6G$1.Q0
- net N$66: now also R42.2; no longer IC6G$1.Q1
- net N$67: now also R43.2; no longer IC6G$1.Q2
- net N$68: now also R44.2; no longer IC6G$1.Q3
- net N$69: now also R45.2; no longer IC6G$1.Q4
- net N$7: now also R4.2; no longer IC1G$1.Q3
- net N$70: now also R46.2; no longer IC6G$1.Q5
- net N$71: now also R47.2; no longer IC6G$1.Q6
- net N$72: now also R48.2; no longer IC6G$1.Q7
- net N$74: now also R49.2; no longer IC7G$1.Q0
- net N$75: now also R50.2; no longer IC7G$1.Q1
- net N$76: now also R51.2; no longer IC7G$1.Q2
- net N$77: now also R52.2; no longer IC7G$1.Q3
- net N$78: now also R53.2; no longer IC7G$1.Q4
- net N$79: now also R54.2; no longer IC7G$1.Q5
- net N$8: now also R5.2; no longer IC1G$1.Q4
- net N$80: now also R55.2; no longer IC7G$1.Q6
- net N$81: now also R56.2; no longer IC7G$1.Q7
- net N$83: now also R57.2; no longer IC8G$1.Q0
- net N$84: now also R58.2; no longer IC8G$1.Q1
- net N$85: now also R59.2; no longer IC8G$1.Q2
- net N$9: now also R6.2; no longer IC1G$1.Q5
Other:
- moved on the sheet: C1, C10, C11, C12, C13, C14, C2, C3, C4, C5, C6, C7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

Commit message: changed out for resistors for more power
Parts:
- removed C10, C11, C12, C13, C14, C9: 100n, rcl:C-EU050-024X044
- removed IC10, IC11, IC9: UDN2981A, uln-udn:UDN2981A
- removed IC12, IC13, IC14: 74HC595N, 74xx-eu:74HC595N
- added Q1, Q10, Q11, Q12, Q13, Q14, Q15, Q16, Q17, Q18, Q19, Q2, Q20, Q21, Q22, Q23, Q24, Q3, Q4, Q5, Q6, Q7, Q8, Q9: S8550D, transistor-pnp:BC558B
Connections:
- removed net N$102: D449.GRN, D450.GRN, D451.GRN, D452.GRN, D453.GRN, D454.GRN, D455.GRN, D456.GRN, D457.GRN, D458.GRN, D459.GRN, D460.GRN, D461.GRN, D462.GRN, D463.GRN, D464.GRN, D465.GRN, D466.GRN, D467.GRN, D468.GRN, D469.GRN, D470.GRN, D471.GRN, D472.GRN, D473.GRN, D474.GRN, D475.GRN, D476.GRN, D477.GRN, D478.GRN, D479.GRN, D480.GRN, D481.GRN, D482.GRN, D483.GRN, D484.GRN, D485.GRN, D486.GRN, D487.GRN, D488.GRN, D489.GRN, D490.GRN, D491.GRN, D492.GRN, D493.GRN, D494.GRN, D495.GRN, D496.GRN, D497.GRN, D498.GRN, D499.GRN, D500.GRN, D501.GRN, D502.GRN, D503.GRN, D504.GRN, D505.GRN, D506.GRN, D507.GRN, D508.GRN, D509.GRN, D510.GRN, D511.GRN, D512.GRN, IC11.O1
- removed net N$105: D257.GRN, D258.GRN, D259.GRN, D260.GRN, D261.GRN, D262.GRN, D263.GRN, D264.GRN, D265.GRN, D266.GRN, D267.GRN, D268.GRN, D269.GRN, D270.GRN, D271.GRN, D272.GRN, D273.GRN, D274.GRN, D275.GRN, D276.GRN, D277.GRN, D278.GRN, D279.GRN, D280.GRN, D281.GRN, D282.GRN, D283.GRN, D284.GRN, D285.GRN, D286.GRN, D287.GRN, D288.GRN, D289.GRN, D290.GRN, D291.GRN, D292.GRN, D293.GRN, D294.GRN, D295.GRN, D296.GRN, D297.GRN, D298.GRN, D299.GRN, D300.GRN, D301.GRN, D302.GRN, D303.GRN, D304.GRN, D305.GRN, D306.GRN, D307.GRN, D308.GRN, D309.GRN, D310.GRN, D311.GRN, D312.GRN, D313.GRN, D314.GRN, D315.GRN, D316.GRN, D317.GRN, D318.GRN, D319.GRN, D320.GRN, IC11.O4
- removed net N$106: IC12A.QG, IC9.I7
- removed net N$108: IC12A.QH*, IC1G$1.DI
- removed net N$110: IC11.I4, IC14A.QD
- removed net N$111: IC10.I1, IC13A.QA
- removed net N$112: IC10.I2, IC13A.QB
- removed net N$113: IC10.I3, IC13A.QC
- removed net N$114: IC10.I4, IC13A.QD
- removed net N$115: IC10.I5, IC13A.QE
- removed net N$116: IC10.I6, IC13A.QF
- removed net N$117: IC10.I7, IC13A.QG
- removed net N$118: IC10.I8, IC13A.QH
- removed net N$119: IC12A.SER, IC13A.QH*
- removed net N$120: IC11.I5, IC14A.QE
- removed net N$121: IC11.I6, IC14A.QF
- removed net N$122: IC11.I7, IC14A.QG
- removed net N$123: IC11.I8, IC14A.QH
- removed net N$124: IC13A.SER, IC14A.QH*
- net GND: no longer C10.2, C11.2, C12.2, C13.2, C14.2, C9.2, IC10.GND, IC11.GND, IC12A.G, IC13A.G, IC14A.G, IC9.GND
- net N$1: now also Q3.C; no longer IC9.O8
- net N$100: now also Q12.C; no longer IC9.O5
- net N$101: now also Q13.E, Q14.E, Q15.E; no longer IC12A.QF, IC9.I6
- net N$103: now also Q19.C; no longer IC11.O2
- net N$104: now also Q16.C; no longer IC11.O3
- net N$107: now also Q16.E, Q17.E, Q18.E; no longer IC12A.QH, IC9.I8
- net N$109: now also Q19.E, Q20.E, Q21.E; no longer IC11.I3, IC14A.QC
- net N$13: no longer IC12A.SCK, IC13A.SCK, IC14A.SCK
- net N$14: no longer IC12A.RCK, IC13A.RCK, IC14A.RCK
- net N$147: now also Q18.C; no longer IC9.O3
- net N$152: now also Q15.C; no longer IC9.O4
- net N$153: now also Q21.C; no longer IC9.O2
- net N$156: now also Q24.C; no longer IC9.O1
- net N$2: now also Q2.C; no longer IC10.O8
- net N$3: now also Q1.C; no longer IC11.O8
- net N$31: now also Q1.E, Q2.E, Q3.E; no longer IC11.I1, IC14A.QA
- net N$32: now also D100.GRN, D101.GRN, D102.GRN, D103.GRN, D104.GRN, D105.GRN, D106.GRN, D107.GRN, D108.GRN, D109.GRN, D110.GRN, D111.GRN, D112.GRN, D113.GRN, D114.GRN, D115.GRN, D116.GRN, D117.GRN, D118.GRN, D119.GRN, D120.GRN, D121.GRN, D122.GRN, D123.GRN, D124.GRN, D125.GRN, D126.GRN, D127.GRN, D128.GRN, D65.GRN, D66.GRN, D67.GRN, D68.GRN, D69.GRN, D70.GRN, D71.GRN, D72.GRN, D73.GRN, D74.GRN, D75.GRN, D76.GRN, D77.GRN, D78.GRN, D79.GRN, D80.GRN, D81.GRN, D82.GRN, D83.GRN, D84.GRN, D85.GRN, D86.GRN, D87.GRN, D88.GRN, D89.GRN, D90.GRN, D91.GRN, D92.GRN, D93.GRN, D94.GRN, D95.GRN, D96.GRN, D97.GRN, D98.GRN, D99.GRN, Q4.C; no longer IC11.I2, IC14A.QB
- net N$46: now also D129.GRN, D130.GRN, D131.GRN, D132.GRN, D133.GRN, D134.GRN, D135.GRN, D136.GRN, D137.GRN, D138.GRN, D139.GRN, D140.GRN, D141.GRN, D142.GRN, D143.GRN, D144.GRN, D145.GRN, D146.GRN, D147.GRN, D148.GRN, D149.GRN, D150.GRN, D151.GRN, D152.GRN, D153.GRN, D154.GRN, D155.GRN, D156.GRN, D157.GRN, D158.GRN, D159.GRN, D160.GRN, D161.GRN, D162.GRN, D163.GRN, D164.GRN, D165.GRN, D166.GRN, D167.GRN, D168.GRN, D169.GRN, D170.GRN, D171.GRN, D172.GRN, D173.GRN, D174.GRN, D175.GRN, D176.GRN, D177.GRN, D178.GRN, D179.GRN, D180.GRN, D181.GRN, D182.GRN, D183.GRN, D184.GRN, D185.GRN, D186.GRN, D187.GRN, D188.GRN, D189.GRN, D190.GRN, D191.GRN, D192.GRN, Q7.C; no longer IC12A.QA, IC9.I1
- net N$47: now also Q7.E, Q8.E, Q9.E; no longer IC12A.QB, IC9.I2
- net N$49: now also Q5.C; no longer IC10.O7
- net N$50: now also Q8.C; no longer IC10.O6
- net N$86: now also Q11.C; no longer IC10.O5
- net N$87: now also Q14.C; no longer IC10.O4
- net N$88: now also Q17.C; no longer IC10.O3
- net N$89: now also Q20.C; no longer IC10.O2
- net N$90: now also Q23.C; no longer IC10.O1
- net N$92: now also D449.GRN, D450.GRN, D451.GRN, D452.GRN, D453.GRN, D454.GRN, D455.GRN, D456.GRN, D457.GRN, D458.GRN, D459.GRN, D460.GRN, D461.GRN, D462.GRN, D463.GRN, D464.GRN, D465.GRN, D466.GRN, D467.GRN, D468.GRN, D469.GRN, D470.GRN, D471.GRN, D472.GRN, D473.GRN, D474.GRN, D475.GRN, D476.GRN, D477.GRN, D478.GRN, D479.GRN, D480.GRN, D481.GRN, D482.GRN, D483.GRN, D484.GRN, D485.GRN, D486.GRN, D487.GRN, D488.GRN, D489.GRN, D490.GRN, D491.GRN, D492.GRN, D493.GRN, D494.GRN, D495.GRN, D496.GRN, D497.GRN, D498.GRN, D499.GRN, D500.GRN, D501.GRN, D502.GRN, D503.GRN, D504.GRN, D505.GRN, D506.GRN, D507.GRN, D508.GRN, D509.GRN, D510.GRN, D511.GRN, D512.GRN, Q22.C; no longer D129.GRN, D130.GRN, D131.GRN, D132.GRN, D133.GRN, D134.GRN, D135.GRN, D136.GRN, D137.GRN, D138.GRN, D139.GRN, D140.GRN, D141.GRN, D142.GRN, D143.GRN, D144.GRN, D145.GRN, D146.GRN, D147.GRN, D148.GRN, D149.GRN, D150.GRN, D151.GRN, D152.GRN, D153.GRN, D154.GRN, D155.GRN, D156.GRN, D157.GRN, D158.GRN, D159.GRN, D160.GRN, D161.GRN, D162.GRN, D163.GRN, D164.GRN, D165.GRN, D166.GRN, D167.GRN, D168.GRN, D169.GRN, D170.GRN, D171.GRN, D172.GRN, D173.GRN, D174.GRN, D175.GRN, D176.GRN, D177.GRN, D178.GRN, D179.GRN, D180.GRN, D181.GRN, D182.GRN, D183.GRN, D184.GRN, D185.GRN, D186.GRN, D187.GRN, D188.GRN, D189.GRN, D190.GRN, D191.GRN, D192.GRN, IC11.O6
- net N$93: now also D193.GRN, D194.GRN, D195.GRN, D196.GRN, D197.GRN, D198.GRN, D199.GRN, D200.GRN, D201.GRN, D202.GRN, D203.GRN, D204.GRN, D205.GRN, D206.GRN, D207.GRN, D208.GRN, D209.GRN, D210.GRN, D211.GRN, D212.GRN, D213.GRN, D214.GRN, D215.GRN, D216.GRN, D217.GRN, D218.GRN, D219.GRN, D220.GRN, D221.GRN, D222.GRN, D223.GRN, D224.GRN, D225.GRN, D226.GRN, D227.GRN, D228.GRN, D229.GRN, D230.GRN, D231.GRN, D232.GRN, D233.GRN, D234.GRN, D235.GRN, D236.GRN, D237.GRN, D238.GRN, D239.GRN, D240.GRN, D241.GRN, D242.GRN, D243.GRN, D244.GRN, D245.GRN, D246.GRN, D247.GRN, D248.GRN, D249.GRN, D250.GRN, D251.GRN, D252.GRN, D253.GRN, D254.GRN, D255.GRN, D256.GRN, Q10.C; no longer D100.GRN, D101.GRN, D102.GRN, D103.GRN, D104.GRN, D105.GRN, D106.GRN, D107.GRN, D108.GRN, D109.GRN, D110.GRN, D111.GRN, D112.GRN, D113.GRN, D114.GRN, D115.GRN, D116.GRN, D117.GRN, D118.GRN, D119.GRN, D120.GRN, D121.GRN, D122.GRN, D123.GRN, D124.GRN, D125.GRN, D126.GRN, D127.GRN, D128.GRN, D65.GRN, D66.GRN, D67.GRN, D68.GRN, D69.GRN, D70.GRN, D71.GRN, D72.GRN, D73.GRN, D74.GRN, D75.GRN, D76.GRN, D77.GRN, D78.GRN, D79.GRN, D80.GRN, D81.GRN, D82.GRN, D83.GRN, D84.GRN, D85.GRN, D86.GRN, D87.GRN, D88.GRN, D89.GRN, D90.GRN, D91.GRN, D92.GRN, D93.GRN, D94.GRN, D95.GRN, D96.GRN, D97.GRN, D98.GRN, D99.GRN, IC11.O7
- net N$94: now also Q4.E, Q5.E, Q6.E; no longer IC12A.QC, IC9.I3
- net N$95: now also Q6.C; no longer IC9.O7
- net N$96: now also Q10.E, Q11.E, Q12.E; no longer IC12A.QD, IC9.I4
- net N$97: now also Q9.C; no longer IC9.O6
- net N$98: now also Q22.E, Q23.E, Q24.E; no longer D193.GRN, D194.GRN, D195.GRN, D196.GRN, D197.GRN, D198.GRN, D199.GRN, D200.GRN, D201.GRN, D202.GRN, D203.GRN, D204.GRN, D205.GRN, D206.GRN, D207.GRN, D208.GRN, D209.GRN, D210.GRN, D211.GRN, D212.GRN, D213.GRN, D214.GRN, D215.GRN, D216.GRN, D217.GRN, D218.GRN, D219.GRN, D220.GRN, D221.GRN, D222.GRN, D223.GRN, D224.GRN, D225.GRN, D226.GRN, D227.GRN, D228.GRN, D229.GRN, D230.GRN, D231.GRN, D232.GRN, D233.GRN, D234.GRN, D235.GRN, D236.GRN, D237.GRN, D238.GRN, D239.GRN, D240.GRN, D241.GRN, D242.GRN, D243.GRN, D244.GRN, D245.GRN, D246.GRN, D247.GRN, D248.GRN, D249.GRN, D250.GRN, D251.GRN, D252.GRN, D253.GRN, D254.GRN, D255.GRN, D256.GRN, IC11.O5
- net N$99: now also D257.GRN, D258.GRN, D259.GRN, D260.GRN, D261.GRN, D262.GRN, D263.GRN, D264.GRN, D265.GRN, D266.GRN, D267.GRN, D268.GRN, D269.GRN, D270.GRN, D271.GRN, D272.GRN, D273.GRN, D274.GRN, D275.GRN, D276.GRN, D277.GRN, D278.GRN, D279.GRN, D280.GRN, D281.GRN, D282.GRN, D283.GRN, D284.GRN, D285.GRN, D286.GRN, D287.GRN, D288.GRN, D289.GRN, D290.GRN, D291.GRN, D292.GRN, D293.GRN, D294.GRN, D295.GRN, D296.GRN, D297.GRN, D298.GRN, D299.GRN, D300.GRN, D301.GRN, D302.GRN, D303.GRN, D304.GRN, D305.GRN, D306.GRN, D307.GRN, D308.GRN, D309.GRN, D310.GRN, D311.GRN, D312.GRN, D313.GRN, D314.GRN, D315.GRN, D316.GRN, D317.GRN, D318.GRN, D319.GRN, D320.GRN, Q13.C; no longer IC12A.QE, IC9.I5
- net VCC: no longer C10.1, C11.1, C12.1, C13.1, C14.1, C9.1, IC10.VS, IC11.VS, IC12A.SCL, IC13A.SCL, IC14A.SCL, IC9.VS
